File: HDMI_TAP/FK_HDMI.kicad_sch (KiCad schematic)
At the start: 3 parts, among them J1 HDMI_A, J2 HDMI_A, J3 Screw_Terminal_01x06

Commit message: Add files via upload
Parts:
- J1: value HDMI_A -> HDMI_A_Male
- J2: value HDMI_A -> HDMI_A_Female
Changed lines of the file:
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@@
 			)
 		)
-		(property "Value" "HDMI_A"
+		(property "Value" "HDMI_A_Female"
 			(at 203.2 101.5999 0)
 			(effects
@@
 			)
 		)
-		(property "Value" "HDMI_A"
+		(property "Value" "HDMI_A_Male"
 			(at 99.06 101.5999 0)
 			(effects
